Commit message: docs: update README with project overview, tech stack, and getting started instructions; remove collision definitions from URDF

File: public/data/kuka_lwr/kuka.urdf (robot description, URDF)
Before this commit: robot kuka_lwr, 8 links, 7 joints
Links:
- link calib_kuka_arm_base_link: geometry visual mesh filename=/data/kuka_lwr/meshes_arm/arm_base.stl
- link kuka_arm_1_link: geometry visual mesh filename=/data/kuka_lwr/meshes_arm/arm_segment_a.stl
- link kuka_arm_2_link: geometry visual mesh filename=/data/kuka_lwr/meshes_arm/arm_segment_b.stl
- link kuka_arm_3_link: geometry visual mesh filename=/data/kuka_lwr/meshes_arm/arm_segment_a.stl
- link kuka_arm_4_link: geometry visual mesh filename=/data/kuka_lwr/meshes_arm/arm_segment_b.stl
- link kuka_arm_5_link: geometry visual mesh filename=/data/kuka_lwr/meshes_arm/arm_segment_last.stl
- link kuka_arm_6_link: geometry visual mesh filename=/data/kuka_lwr/meshes_arm/arm_wrist.stl
- link kuka_arm_7_link: geometry visual mesh filename=/data/kuka_lwr/meshes_arm/arm_flanche.stl
